File: _4mm_sleeper/_4mm_sleeper.kicad_pcb (KiCad board)
At the start: 2 copper layers, 10.4 x 30 mm, 0 parts

Commit message: made production files
Other:
- board text added: "OSHW"
- board text removed: "Train-Science.com"
