File: _7mm_sleeper/_7mm_sleeper.kicad_pcb (KiCad board)
At the start: 2 copper layers, 13.4 x 30 mm, 0 parts

Commit message: made production files
Other:
- board text added: "OSHW"
- board text removed: "Train-Science.com"
